Commit message: Checkpoint2

File: description/robot_core.xacro (robot description, xacro)
@@ -48,4 +48,7 @@
         </xacro:inertial_box>
     </link>
+    <gazebo reference="chassis">
+        <material>Gazebo/White</material>
+    </gazebo>
     <!-- WHEEL SECTION -->
     <!-- left wheel joint -->
@@ -73,4 +76,7 @@
         </xacro:inertial_cylinder>
     </link>
+    <gazebo reference="left_wheel">
+        <material>Gazebo/Blue</material>
+    </gazebo>
     <!-- right wheel joint -->
     <joint name="right_wheel_joint" type="continuous">
@@ -97,4 +103,7 @@
         </xacro:inertial_cylinder>
     </link>
+    <gazebo reference="right_wheel">
+        <material>Gazebo/Blue</material>
+    </gazebo>
     <!-- caster wheel joint -->
     <joint name="caster_wheel_joint" type="fixed">
@@ -120,3 +129,8 @@
         </xacro:inertial_sphere>
     </link>
+    <gazebo reference="caster_wheel">
+        <material>Gazebo/Black</material>
+        <mu1 value="0.000001"/>
+        <mu2 value="0.000001"/>
+    </gazebo>
 </robot>
