Commit message: Add sensors

File: description/robot.urdf.xacro (robot description, xacro)
@@ -3,3 +3,5 @@
     <xacro:include filename="robot_core.xacro" />
     <xacro:include filename="gazebo_control.xacro"/>
+    <xacro:include filename="lidar.xacro"/>
+    <xacro:include filename="depth_camera.xacro"/>
 </robot>

File: description/robot_core.xacro (robot description, xacro)
@@ -18,4 +18,8 @@
     <material name="black">
         <color rgba="0 0 0 1"/>
+    </material>
+    <!-- red color -->
+    <material>
+        <color rgba="1 0 0 1"/>
     </material>
     <!-- BASE LINK -->
